File: connectors.kicad_sch (KiCad schematic)
At the start: 4 parts, among them J1 Conn_01x09_Male, J2 Conn_01x04_Male, J3 Conn_01x04_Male, J4 Conn_02x03_Odd_Even

Commit message: footprints
Parts:
- J1: footprint (none) -> Connector_PinSocket_2.54mm:PinSocket_1x09_P2.54mm_Vertical
- J2, J3: footprint (none) -> Connector_PinHeader_2.54mm:PinHeader_1x04_P2.54mm_Vertical
- J4: footprint (none) -> Connector_PinSocket_2.54mm:PinSocket_2x03_P2.54mm_Vertical
Changed lines of the file:
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@@
     (property "Reference" "J4" (id 0) (at 120.015 77.47 0))
     (property "Value" "Conn_02x03_Odd_Even" (id 1) (at 120.015 80.01 0))
-    (property "Footprint" "" (id 2) (at 118.745 86.995 0)
+    (property "Footprint" "Connector_PinSocket_2.54mm:PinSocket_2x03_P2.54mm_Vertical" (id 2) (at 118.745 86.995 0)
       (effects (font (size 1.27 1.27)) hide)
     )
@@
     (property "Reference" "J3" (id 0) (at 118.11 53.34 0))
     (property "Value" "Conn_01x04_Male" (id 1) (at 118.11 55.88 0))
-    (property "Footprint" "" (id 2) (at 117.475 60.96 0)
+    (property "Footprint" "Connector_PinHeader_2.54mm:PinHeader_1x04_P2.54mm_Vertical" (id 2) (at 117.475 60.96 0)
       (effects (font (size 1.27 1.27)) hide)
     )
@@
     (property "Reference" "J1" (id 0) (at 90.17 80.01 0))
     (property "Value" "Conn_01x09_Male" (id 1) (at 90.17 82.55 0))
-    (property "Footprint" "" (id 2) (at 89.535 95.885 0)
+    (property "Footprint" "Connector_PinSocket_2.54mm:PinSocket_1x09_P2.54mm_Vertical" (id 2) (at 89.535 95.885 0)
       (effects (font (size 1.27 1.27)) hide)
     )
@@
     (property "Reference" "J2" (id 0) (at 90.805 54.61 0))
     (property "Value" "Conn_01x04_Male" (id 1) (at 90.805 57.15 0))
-    (property "Footprint" "" (id 2) (at 90.17 62.865 0)
+    (property "Footprint" "Connector_PinHeader_2.54mm:PinHeader_1x04_P2.54mm_Vertical" (id 2) (at 90.17 62.865 0)
       (effects (font (size 1.27 1.27)) hide)
     )

Commit message: finished wiring
Connections:
- net MISO: now reaches J4.1 (Pin_1)
- net Vcc: now reaches J4.2 (Pin_2)
- net Vcc: now also J1.9 (Pin_9), J2.2 (Pin_2), J3.2 (Pin_2)
- net SCK: now reaches J4.3 (Pin_3)
- net SCK: now also J2.4 (Pin_4)
- net MOSI: now reaches J4.4 (Pin_4)
- net RESET: now reaches J4.5 (Pin_5)
- net GND: now reaches J4.6 (Pin_6)
- net GND: now also J1.8 (Pin_8), J2.1 (Pin_1), J3.1 (Pin_1)
- net RX: now reaches J3.3 (Pin_3)
- net TX: now reaches J3.4 (Pin_4)
- net D2: now reaches J1.1 (Pin_1)
- net D3: now reaches J1.2 (Pin_2)
- net D4: now reaches J1.3 (Pin_3)
- net D5: now reaches J1.4 (Pin_4)
- net D6: now reaches J1.5 (Pin_5)
- net D7: now reaches J1.6 (Pin_6)
- net D8: now reaches J1.7 (Pin_7)
- net SDA: now reaches J2.3 (Pin_3)
Changed lines of the file:
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@@
 (kicad_sch (version 20211123) (generator eeschema)
   (paper "A4")
+  (hierarchical_label "Vcc" (shape passive) (at 122.555 60.96 0)
+    (effects (font (size 1.27 1.27)) (justify left))
+  )
+  (hierarchical_label "D7" (shape bidirectional) (at 94.615 98.425 0)
+    (effects (font (size 1.27 1.27)) (justify left))
+  )
+  (hierarchical_label "D6" (shape bidirectional) (at 94.615 95.885 0)
+    (effects (font (size 1.27 1.27)) (justify left))
+  )
+  (hierarchical_label "SCK" (shape passive) (at 113.665 86.995 180)
+    (effects (font (size 1.27 1.27)) (justify right))
+  )
+  (hierarchical_label "MOSI" (shape input) (at 126.365 86.995 0)
+    (effects (font (size 1.27 1.27)) (justify left))
+  )
+  (hierarchical_label "TX" (shape output) (at 122.555 66.04 0)
+    (effects (font (size 1.27 1.27)) (justify left))
+  )
+  (hierarchical_label "GND" (shape passive) (at 94.615 103.505 0)
+    (effects (font (size 1.27 1.27)) (justify left))
+  )
+  (hierarchical_label "GND" (shape passive) (at 122.555 58.42 0)
+    (effects (font (size 1.27 1.27)) (justify left))
+  )
+  (hierarchical_label "RX" (shape input) (at 122.555 63.5 0)
+    (effects (font (size 1.27 1.27)) (justify left))
+  )
+  (hierarchical_label "Vcc" (shape passive) (at 94.615 106.045 0)
+    (effects (font (size 1.27 1.27)) (justify left))
+  )
+  (hierarchical_label "Vcc" (shape passive) (at 95.25 62.865 0)
+    (effects (font (size 1.27 1.27)) (justify left))
+  )
+  (hierarchical_label "SCK" (shape passive) (at 95.25 67.945 0)
+    (effects (font (size 1.27 1.27)) (justify left))
+  )
+  (hierarchical_label "MISO" (shape output) (at 113.665 84.455 180)
+    (effects (font (size 1.27 1.27)) (justify right))
+  )
+  (hierarchical_label "SDA" (shape bidirectional) (at 95.25 65.405 0)
+    (effects (font (size 1.27 1.27)) (justify left))
+  )
+  (hierarchical_label "RESET" (shape passive) (at 113.665 89.535 180)
+    (effects (font (size 1.27 1.27)) (justify right))
+  )
+  (hierarchical_label "Vcc" (shape passive) (at 126.365 84.455 0)
+    (effects (font (size 1.27 1.27)) (justify left))
+  )
+  (hierarchical_label "GND" (shape passive) (at 126.365 89.535 0)
+    (effects (font (size 1.27 1.27)) (justify left))
+  )
+  (hierarchical_label "D5" (shape bidirectional) (at 94.615 93.345 0)
+    (effects (font (size 1.27 1.27)) (justify left))
+  )
+  (hierarchical_label "D3" (shape bidirectional) (at 94.615 88.265 0)
+    (effects (font (size 1.27 1.27)) (justify left))
+  )
+  (hierarchical_label "D2" (shape bidirectional) (at 94.615 85.725 0)
+    (effects (font (size 1.27 1.27)) (justify left))
+  )
+  (hierarchical_label "D4" (shape bidirectional) (at 94.615 90.805 0)
+    (effects (font (size 1.27 1.27)) (justify left))
+  )
+  (hierarchical_label "GND" (shape passive) (at 95.25 60.325 0)
+    (effects (font (size 1.27 1.27)) (justify left))
+  )
+  (hierarchical_label "D8" (shape bidirectional) (at 94.615 100.965 0)
+    (effects (font (size 1.27 1.27)) (justify left))
+  )
   (symbol (lib_id "Connector_Generic:Conn_02x03_Odd_Even") (at 118.745 86.995 0) (unit 1)
     (in_bom yes) (on_board yes)
@@
   )
   (symbol (lib_id "Connector:Conn_01x09_Male") (at 89.535 95.885 0) (unit 1)
-    (in_bom yes) (on_board yes) (fields_autoplaced)
+    (in_bom yes) (on_board yes)
     (property "Reference" "J1" (id 0) (at 90.17 80.01 0))
     (property "Value" "Conn_01x09_Male" (id 1) (at 90.17 82.55 0))
@@
       (effects (font (size 1.27 1.27)) hide)
     )
-    (property "Purpose" "GPIO Header" (id 4) (at 89.535 95.885 0))
+    (property "Purpose" "GPIO Header" (id 4) (at 91.44 109.855 0))
     (pin "1")
     (pin "2")
